File: kicad/STM32L0LoraTx/STM32L0LoraTx-black-labels.kicad_pcb (KiCad board)
At the start: 2 copper layers, 58.8 x 23 mm, 22 parts, among them J1 Conn_01x04, J2 Conn_01x06, J3 Barrel_Jack, J4 Conn_01x06, J5 Barrel_Jack, J6 Conn_01x02, U1 STM32L011F4Px, U2 RFM95W-868S2

Commit message: add bme280 support
Parts:
- J2, J4: value Conn_01x06 -> Conn_01x06_Female
Routing:
- net Net-(R3-Pad2): track 2.06 -> 0.00 mm
